Commit message: fix

File: mg400_description/urdf/mg400_description.urdf.xacro (robot description, xacro)
@@ -1,27 +1,61 @@
 <?xml version="1.0" encoding="utf-8"?>
-<robot xmlns:xacro="http://ros.org/wiki/xacro" name="mg400">
+<robot
+    xmlns:xacro="http://ros.org/wiki/xacro"
+    name="mg400">
   <!-- Import Rviz colors -->
   <xacro:include filename="$(find mg400_description)/xacro/materials.xacro" />
   <!-- constants -->
-  <xacro:include filename="$(find mg400_description)/xacro/constants.xacro" ns="const" />
+  <xacro:include
+      filename="$(find mg400_description)/xacro/constants.xacro"
+      ns="const" />
   <!-- Base path for meshes -->
-  <xacro:property name="BASE_PATH" value="mg400_description/meshes" />
-  <xacro:property name="MESH_BASE_LINK" value="${BASE_PATH}/base_link.stl" />
-  <xacro:property name="MESH_LINK_1" value="${BASE_PATH}/link1.stl" />
-  <xacro:property name="MESH_LINK_2_1" value="${BASE_PATH}/link2_1.stl" />
-  <xacro:property name="MESH_LINK_2_2" value="${BASE_PATH}/link2_2.stl" />
-  <xacro:property name="MESH_LINK_3_1" value="${BASE_PATH}/link3_1.stl" />
-  <xacro:property name="MESH_LINK_3_2" value="${BASE_PATH}/link3_2.stl" />
-  <xacro:property name="MESH_LINK_4_1" value="${BASE_PATH}/link4_1.stl" />
-  <xacro:property name="MESH_LINK_4_2" value="${BASE_PATH}/link4_2.stl" />
-  <xacro:property name="MESH_LINK_5" value="${BASE_PATH}/link5.stl" />
+  <xacro:property
+      name="BASE_PATH"
+      value="mg400_description/meshes" />
+  <xacro:property
+      name="MESH_BASE_LINK"
+      value="${BASE_PATH}/base_link.stl" />
+  <xacro:property
+      name="MESH_LINK_1"
+      value="${BASE_PATH}/link1.stl" />
+  <xacro:property
+      name="MESH_LINK_2_1"
+      value="${BASE_PATH}/link2_1.stl" />
+  <xacro:property
+      name="MESH_LINK_2_2"
+      value="${BASE_PATH}/link2_2.stl" />
+  <xacro:property
+      name="MESH_LINK_3_1"
+      value="${BASE_PATH}/link3_1.stl" />
+  <xacro:property
+      name="MESH_LINK_3_2"
+      value="${BASE_PATH}/link3_2.stl" />
+  <xacro:property
+      name="MESH_LINK_4_1"
+      value="${BASE_PATH}/link4_1.stl" />
+  <xacro:property
+      name="MESH_LINK_4_2"
+      value="${BASE_PATH}/link4_2.stl" />
+  <xacro:property
+      name="MESH_LINK_5"
+      value="${BASE_PATH}/link5.stl" />
   <link name="base_link">
     <inertial>
-      <origin xyz="0.000600637001378879 -2.53487071137343E-07 0.0560927888040551" rpy="0 0 0" />
+      <origin
+          xyz="0.000600637001378879 -2.53487071137343E-07 0.0560927888040551"
+          rpy="0 0 0" />
       <mass value="3.62164811695094" />
-      <inertia ixx="0.0126582175296405" ixy="6.66832041405407E-08" ixz="-3.52548281362717E-06" iyy="0.0145891535260188" iyz="5.15901657460475E-08" izz="0.0195045116656827" />
-    </inertial>
-    <visual>
-      <origin xyz="0 0 0" rpy="0 0 0" />
+      <inertia
+          ixx="0.0126582175296405"
+          ixy="6.66832041405407E-08"
+          ixz="-3.52548281362717E-06"
+          iyy="0.0145891535260188"
+          iyz="5.15901657460475E-08"
+          izz="0.0195045116656827" />
+    </inertial>
+    <visual>
+      <origin
+          xyz="0 0 0"
+          rpy="0 0 0" />
       <geometry>
         <mesh filename="package://${MESH_BASE_LINK}" />
@@ -30,5 +64,7 @@
     </visual>
     <collision>
-      <origin xyz="0 0 0" rpy="0 0 0" />
+      <origin
+          xyz="0 0 0"
+          rpy="0 0 0" />
       <geometry>
         <mesh filename="package://${MESH_BASE_LINK}" />
@@ -38,10 +74,20 @@
   <link name="link1">
     <inertial>
-      <origin xyz="-0.0046209286967387 -6.88107982318643E-05 0.0709919358465827" rpy="0 0 0" />
+      <origin
+          xyz="-0.0046209286967387 -6.88107982318643E-05 0.0709919358465827"
+          rpy="0 0 0" />
       <mass value="1.77056222753813" />
-      <inertia ixx="0.00605885293080088" ixy="0.000156081820035162" ixz="-0.00021785654850453" iyy="0.00579381982249127" iyz="6.20876898015621E-05" izz="0.00741058257251941" />
-    </inertial>
-    <visual>
-      <origin xyz="0 0 0" rpy="0 0 0" />
+      <inertia
+          ixx="0.00605885293080088"
+          ixy="0.000156081820035162"
+          ixz="-0.00021785654850453"
+          iyy="0.00579381982249127"
+          iyz="6.20876898015621E-05"
+          izz="0.00741058257251941" />
+    </inertial>
+    <visual>
+      <origin
+          xyz="0 0 0"
+          rpy="0 0 0" />
       <geometry>
         <mesh filename="package://${MESH_LINK_1}" />
@@ -50,5 +96,7 @@
     </visual>
     <collision>
-      <origin xyz="0 0 0" rpy="0 0 0" />
+      <origin
+          xyz="0 0 0"
+          rpy="0 0 0" />
       <geometry>
         <mesh filename="package://${MESH_LINK_1}" />
@@ -56,19 +104,37 @@
     </collision>
   </link>
-  <joint name="j1" type="revolute">
-    <origin xyz="${-5.0 * const.SCALE_MM} 0 ${109 * const.SCALE_MM}" rpy="0 0 0" />
+  <joint
+      name="j1"
+      type="revolute">
+    <origin
+        xyz="${-5.0 * const.SCALE_MM} 0 ${109 * const.SCALE_MM}"
+        rpy="0 0 0" />
     <parent link="base_link" />
     <child link="link1" />
     <axis xyz="0 0 1" />
-    <limit lower="${-180.0 * const.TO_RADIAN}" upper="${180.0 * const.TO_RADIAN}" effort="0" velocity="0" />
+    <limit
+        lower="${-180.0 * const.TO_RADIAN}"
+        upper="${180.0 * const.TO_RADIAN}"
+        effort="0"
+        velocity="0" />
   </joint>
   <link name="link2_1">
     <inertial>
-      <origin xyz="-0.00321788524756698 0.0352926570826593 0.0596131328734945" rpy="0 0 0" />
+      <origin
+          xyz="-0.00321788524756698 0.0352926570826593 0.0596131328734945"
+          rpy="0 0 0" />
       <mass value="0.0866115884541459" />
-      <inertia ixx="0.000338551627157209" ixy="-2.78858228577314E-09" ixz="1.05212346076681E-05" iyy="0.000307789653713489" iyz="-1.36109590152488E-06" izz="3.89949940178023E-05" />
-    </inertial>
-    <visual>
-      <origin xyz="0 0 0" rpy="0 0 0" />
+      <inertia
+          ixx="0.000338551627157209"
+          ixy="-2.78858228577314E-09"
+          ixz="1.05212346076681E-05"
+          iyy="0.000307789653713489"
+          iyz="-1.36109590152488E-06"
+          izz="3.89949940178023E-05" />
+    </inertial>
+    <visual>
+      <origin
+          xyz="0 0 0"
+          rpy="0 0 0" />
       <geometry>
         <mesh filename="package://${MESH_LINK_2_1}" />
@@ -77,5 +143,7 @@
     </visual>
     <collision>
-      <origin xyz="0 0 0" rpy="0 0 0" />
+      <origin
+          xyz="0 0 0"
+          rpy="0 0 0" />
       <geometry>
         <mesh filename="package://${MESH_LINK_2_1}" />
@@ -83,19 +151,37 @@
     </collision>
   </link>
-  <joint name="j2_1" type="revolute">
-    <origin xyz="0.0435007595118091 -0.0357748756218899 0.118995682641123" rpy="0 0 0" />
+  <joint
+      name="j2_1"
+      type="revolute">
+    <origin
+        xyz="0.0435007595118091 -0.0357748756218899 0.118995682641123"
+        rpy="0 0 0" />
     <parent link="link1" />
     <child link="link2_1" />
     <axis xyz="0 1 0" />
-    <limit lower="-3.14" upper="3.14" effort="0" velocity="0" />
+    <limit
+        lower="-3.14"
+        upper="3.14"
+        effort="0"
+        velocity="0" />
   </joint>
   <link name="link3_1">
     <inertial>
-      <origin xyz="0.0821679417596488 0.000113044685842874 -0.00333758753063973" rpy="0 0 0" />
+      <origin
+          xyz="0.0821679417596488 0.000113044685842874 -0.00333758753063973"
+          rpy="0 0 0" />
       <mass value="0.0375214831045061" />
-      <inertia ixx="2.54761091812684E-06" ixy="3.73102654491378E-07" ixz="-2.02625705871199E-06" iyy="0.000164234314177935" iyz="-1.44731096825347E-08" izz="0.000164331500854172" />
-    </inertial>
-    <visual>
-      <origin xyz="0 0 0" rpy="0 0 0" />
+      <inertia
+          ixx="2.54761091812684E-06"
+          ixy="3.73102654491378E-07"
+          ixz="-2.02625705871199E-06"
+          iyy="0.000164234314177935"
+          iyz="-1.44731096825347E-08"
+          izz="0.000164331500854172" />
+    </inertial>
+    <visual>
+      <origin
+          xyz="0 0 0"
+          rpy="0 0 0" />
       <geometry>
         <mesh filename="package://${MESH_LINK_3_1}" />
@@ -104,5 +190,7 @@
     </visual>
     <collision>
-      <origin xyz="0 0 0" rpy="0 0 0" />
+      <origin
+          xyz="0 0 0"
+          rpy="0 0 0" />
       <geometry>
         <mesh filename="package://${MESH_LINK_3_1}" />
@@ -110,19 +198,37 @@
     </collision>
   </link>
-  <joint name="j3_1" type="revolute">
-    <origin xyz="-0.0010512570171516 0.0357748756218898 0.175001164344716" rpy="0 0 0" />
+  <joint
+      name="j3_1"
+      type="revolute">
+    <origin
+        xyz="-0.0010512570171516 0.0357748756218898 0.175001164344716"
+        rpy="0 0 0" />
     <parent link="link2_1" />
     <child link="link3_1" />
     <axis xyz="0 1 0" />
-    <limit lower="-3.14" upper="3.14" effort="0" velocity="0" />
+    <limit
+        lower="-3.14"
+        upper="3.14"
+        effort="0"
+        velocity="0" />
   </joint>
   <link name="link4_1">
     <inertial>
-      <origin xyz="0.0387878182928232 0.0170848333998282 -0.0024610990490942" rpy="0 0 0" />
+      <origin
+          xyz="0.0387878182928232 0.0170848333998282 -0.0024610990490942"
+          rpy="0 0 0" />
       <mass value="0.0628979533925801" />
-      <inertia ixx="4.78483605712844E-05" ixy="1.42081909356751E-07" ixz="8.32917079044309E-06" iyy="5.42362047732042E-05" iyz="-2.90608446019989E-08" izz="3.36120409842199E-05" />
-    </inertial>
-    <visual>
-      <origin xyz="0 0 0" rpy="0 0 0" />
+      <inertia
+          ixx="4.78483605712844E-05"
+          ixy="1.42081909356751E-07"
+          ixz="8.32917079044309E-06"
+          iyy="5.42362047732042E-05"
+          iyz="-2.90608446019989E-08"
+          izz="3.36120409842199E-05" />
+    </inertial>
+    <visual>
+      <origin
+          xyz="0 0 0"
+          rpy="0 0 0" />
       <geometry>
         <mesh filename="package://${MESH_LINK_4_1}" />
@@ -131,5 +237,7 @@
     </visual>
     <collision>
-      <origin xyz="0 0 0" rpy="0 0 0" />
+      <origin
+          xyz="0 0 0"
+          rpy="0 0 0" />
       <geometry>
         <mesh filename="package://${MESH_LINK_4_1}" />
@@ -137,19 +245,37 @@
     </collision>
   </link>
-  <joint name="j4_1" type="revolute">
-    <origin xyz="0.174969784055705 -0.0170000000000335 0.00325187137614585" rpy="0 0 0" />
+  <joint
+      name="j4_1"
+      type="revolute">
+    <origin
+        xyz="0.174969784055705 -0.0170000000000335 0.00325187137614585"
+        rpy="0 0 0" />
     <parent link="link3_1" />
     <child link="link4_1" />
     <axis xyz="0 1 0" />
-    <limit lower="-3.14" upper="3.14" effort="0" velocity="0" />
+    <limit
+        lower="-3.14"
+        upper="3.14"
+        effort="0"
+        velocity="0" />
   </joint>
   <link name="link5">
     <inertial>
-      <origin xyz="4.24246458685662E-07 3.08507851181768E-14 -0.0349688816440933" rpy="0 0 0" />
+      <origin
+          xyz="4.24246458685662E-07 3.08507851181768E-14 -0.0349688816440933"
+          rpy="0 0 0" />
       <mass value="0.0965276919819365" />
-      <inertia ixx="4.98589992160928E-05" ixy="-1.534865545378E-12" ixz="3.46424449605658E-10" iyy="4.98589881725446E-05" iyz="-5.64890953414983E-17" izz="2.130463008359E-05" />
-    </inertial>
-    <visual>
-      <origin xyz="0 0 0" rpy="0 0 0" />
+      <inertia
+          ixx="4.98589992160928E-05"
+          ixy="-1.534865545378E-12"
+          ixz="3.46424449605658E-10"
+          iyy="4.98589881725446E-05"
+          iyz="-5.64890953414983E-17"
+          izz="2.130463008359E-05" />
+    </inertial>
+    <visual>
+      <origin
+          xyz="0 0 0"
+          rpy="0 0 0" />
       <geometry>
         <mesh filename="package://${MESH_LINK_5}" />
@@ -158,5 +284,7 @@
     </visual>
     <collision>
-      <origin xyz="0 0 0" rpy="0 0 0" />
+      <origin
+          xyz="0 0 0"
+          rpy="0 0 0" />
       <geometry>
         <mesh filename="package://${MESH_LINK_5}" />
@@ -164,6 +292,10 @@
     </collision>
   </link>
-  <joint name="j5_1" type="fixed">
-    <origin xyz="0.0659996239003897 0.0170000000000371 0.031000800715573" rpy="0 0 0" />
+  <joint
+      name="j5_1"
+      type="fixed">
+    <origin
+        xyz="0.0659996239003897 0.0170000000000371 0.031000800715573"
+        rpy="0 0 0" />
     <parent link="link4_1" />
     <child link="link5" />
@@ -172,32 +304,58 @@
   <link name="end_effector_shaft">
     <visual>
-      <origin xyz="0 0 0" rpy="0 0 0" />
-      <geometry>
-        <cylinder radius="${4.0 * const.SCALE_MM}" length="${15.0 * const.SCALE_MM}" />
+      <origin
+          xyz="0 0 0"
+          rpy="0 0 0" />
+      <geometry>
+        <cylinder
+            radius="${4.0 * const.SCALE_MM}"
+            length="${15.0 * const.SCALE_MM}" />
       </geometry>
       <material name="red" />
     </visual>
     <collision>
-      <origin xyz="0 0 0" rpy="0 0 0" />
-      <geometry>
-        <cylinder radius="${4.0 * const.SCALE_MM}" length="${15.0 * const.SCALE_MM}" />
-      </geometry>
-    </collision>
-  </link>
-  <joint name="j5" type="revolute">
-    <origin xyz="0 0 ${-70.0 * const.SCALE_MM}" rpy="0 0 0" />
+      <origin
+          xyz="0 0 0"
+          rpy="0 0 0" />
+      <geometry>
+        <cylinder
+            radius="${4.0 * const.SCALE_MM}"
+            length="${15.0 * const.SCALE_MM}" />
+      </geometry>
+    </collision>
+  </link>
+  <joint
+      name="j5"
+      type="revolute">
+    <origin
+        xyz="0 0 ${-70.0 * const.SCALE_MM}"
+        rpy="0 0 0" />
     <parent link="link5" />
     <child link="end_effector_shaft" />
     <axis xyz="0 0 1" />
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