Commit message: set physical parameter to urdf

File: mg400_description/urdf/mg400.xacro (robot description, xacro)
@@ -68,4 +68,12 @@
         </geometry>
       </visual>
+      <collision>
+        <origin
+            xyz="0 0 0"
+            rpy="0 0 0" />
+        <geometry>
+          <mesh filename="package://${MESH_BASE_LINK}" />
+        </geometry>
+      </collision>
     </link>
     <link name="${prefix}mg400_origin_link" />
@@ -92,4 +100,12 @@
         </geometry>
       </visual>
+      <collision>
+        <origin
+            xyz="0 0 0"
+            rpy="0 0 0" />
+        <geometry>
+          <mesh filename="package://${MESH_LINK_1}" />
+        </geometry>
+      </collision>
     </link>
     <link name="${prefix}mg400_link2_1">
@@ -115,4 +131,12 @@
         </geometry>
       </visual>
+      <collision>
+        <origin
+            xyz="0 0 0"
+            rpy="0 0 0" />
+        <geometry>
+          <mesh filename="package://${MESH_LINK_2_1}" />
+        </geometry>
+      </collision>
     </link>
     <link name="${prefix}mg400_link2_2">
@@ -138,4 +162,12 @@
         </geometry>
       </visual>
+      <collision>
+        <origin
+            xyz="0 0 0"
+            rpy="0 0 0" />
+        <geometry>
+          <mesh filename="package://${MESH_LINK_2_2}" />
+        </geometry>
+      </collision>
     </link>
     <link name="${prefix}mg400_link3_1">
@@ -161,4 +193,12 @@
         </geometry>
       </visual>
+      <collision>
+        <origin
+            xyz="0 0 0"
+            rpy="0 0 0" />
+        <geometry>
+          <mesh filename="package://${MESH_LINK_3_1}" />
+        </geometry>
+      </collision>
     </link>
     <link name="${prefix}mg400_link3_2">
@@ -184,4 +224,12 @@
         </geometry>
       </visual>
+      <collision>
+        <origin
+            xyz="0 0 0"
+            rpy="0 0 0" />
+        <geometry>
+          <mesh filename="package://${MESH_LINK_3_2}" />
+        </geometry>
+      </collision>
     </link>
     <link name="${prefix}mg400_link4_1">
@@ -207,4 +255,12 @@
         </geometry>
       </visual>
+      <collision>
+        <origin
+            xyz="0 0 0"
+            rpy="0 0 0" />
+        <geometry>
+          <mesh filename="package://${MESH_LINK_4_1}" />
+        </geometry>
+      </collision>
     </link>
     <link name="${prefix}mg400_link4_2">
@@ -230,6 +286,27 @@
         </geometry>
       </visual>
+      <collision>
+        <origin
+            xyz="0 0 0"
+            rpy="0 0 0" />
+        <geometry>
+          <mesh filename="package://${MESH_LINK_4_2}" />
+        </geometry>
+      </collision>
     </link>
     <link name="${prefix}mg400_link4_3">
+      <inertial>
+        <origin
+            xyz="${3.174 * const.SCALE_MM} 0.0 ${-28.198 * const.SCALE_MM}"
+            rpy="0 0 0" />
+        <mass value="0.01907" />
+        <inertia
+            ixx="3.28164E-05"
+            ixy="3.15E-10"
+            ixz="2.42378E-06"
+            iyy="3.17191E-05"
+            iyz="-1.27E-10"
+            izz="1.08143E-05" />
+      </inertial>
       <visual>
         <origin
@@ -240,4 +317,12 @@
         </geometry>
       </visual>
+      <collision>
+        <origin
+            xyz="0 0 0"
+            rpy="0 0 0" />
+        <geometry>
+          <mesh filename="package://${MESH_LINK_4_3}" />
+        </geometry>
+      </collision>
     </link>
     <link name="${prefix}mg400_link5">
@@ -263,4 +348,12 @@
         </geometry>
       </visual>
+      <collision>
+        <origin
+            xyz="0 0 0"
+            rpy="0 0 0" />
+        <geometry>
+          <mesh filename="package://${MESH_LINK_5}" />
+        </geometry>
+      </collision>
     </link>
     <link name="${prefix}mg400_end_effector_shaft">
@@ -276,9 +369,7 @@
         <origin
             xyz="0 0 0"
-            rpy="0 0 0" />
-        <geometry>
-          <cylinder
-              radius="${4.0 * const.SCALE_MM}"
-              length="${15.0 * const.SCALE_MM}" />
+            rpy="${180.0 * const.TO_RADIAN} 0 0" />
+        <geometry>
+          <mesh filename="package://${MESH_SHAFT}" />
         </geometry>
       </collision>

Commit message: fix urdf shaft -> flange

File: mg400_description/urdf/mg400.xacro (robot description, xacro)
@@ -40,6 +40,6 @@
       value="${BASE_PATH}/link5.dae" />
   <xacro:property
-      name="MESH_SHAFT"
-      value="${BASE_PATH}/shaft.dae" />
+      name="MESH_FLANGE"
+      value="${BASE_PATH}/flange.dae" />
   <xacro:macro
       name="mg400"
@@ -357,19 +357,32 @@
       </collision>
     </link>
-    <link name="${prefix}mg400_end_effector_shaft">
-      <visual>
-        <origin
-            xyz="0 0 0"
-            rpy="${180.0 * const.TO_RADIAN} 0 0" />
-        <geometry>
-          <mesh filename="package://${MESH_SHAFT}" />
-        </geometry>
-      </visual>
-      <collision>
-        <origin
-            xyz="0 0 0"
-            rpy="${180.0 * const.TO_RADIAN} 0 0" />
-        <geometry>
-          <mesh filename="package://${MESH_SHAFT}" />
+    <link name="${prefix}mg400_end_effector_flange">
+      <inertial>
+        <origin
+            xyz="0 0 5.0e-3"
+            rpy="0 0 0" />
+        <mass value="24.0e-3" />
+        <inertia
+            ixx="2.058-6"
+            ixy="0.0"
+            ixz="0.0"
+            iyy="2.058-6"
+            iyz="0.0"
+            izz="3.335e-6" />
+      </inertial>
+      <visual>
+        <origin
+            xyz="0 0 0"
+            rpy="0 0 0" />
+        <geometry>
+          <mesh filename="package://${MESH_FLANGE}" />
+        </geometry>
+      </visual>
+      <collision>
+        <origin
+            xyz="0 0 0"
+            rpy="0 0 0" />
+        <geometry>
+          <mesh filename="package://${MESH_FLANGE}" />
         </geometry>
       </collision>
@@ -519,5 +532,5 @@
         type="revolute">
       <origin
-          xyz="0 0 ${-70.0 * const.SCALE_MM}"
+          xyz="0 0 ${(-70.0 - 14.0) * const.SCALE_MM}"
           rpy="0 0 0" />
       <parent link="${prefix}mg400_link5" />

Commit message: fix joint bug

File: mg400_description/urdf/mg400.xacro (robot description, xacro)
@@ -535,5 +535,5 @@
           rpy="0 0 0" />
       <parent link="${prefix}mg400_link5" />
-      <child link="${prefix}mg400_end_effector_shaft" />
+      <child link="${prefix}mg400_end_effector_flange" />
       <axis xyz="0 0 1" />
       <limit

Commit message: Features/flange (#89)
* fix urdf shaft -> flange

* add flange meshes

* fix joint bug

File: mg400_description/urdf/mg400.xacro (robot description, xacro)
@@ -40,6 +40,6 @@
       value="${BASE_PATH}/link5.dae" />
   <xacro:property
-      name="MESH_SHAFT"
-      value="${BASE_PATH}/shaft.dae" />
+      name="MESH_FLANGE"
+      value="${BASE_PATH}/flange.dae" />
   <xacro:macro
       name="mg400"
@@ -357,19 +357,32 @@
       </collision>
     </link>
-    <link name="${prefix}mg400_end_effector_shaft">
-      <visual>
-        <origin
-            xyz="0 0 0"
-            rpy="${180.0 * const.TO_RADIAN} 0 0" />
-        <geometry>
-          <mesh filename="package://${MESH_SHAFT}" />
-        </geometry>
-      </visual>
-      <collision>
-        <origin
-            xyz="0 0 0"
-            rpy="${180.0 * const.TO_RADIAN} 0 0" />
-        <geometry>
-          <mesh filename="package://${MESH_SHAFT}" />
+    <link name="${prefix}mg400_end_effector_flange">
+      <inertial>
+        <origin
+            xyz="0 0 5.0e-3"
+            rpy="0 0 0" />
+        <mass value="24.0e-3" />
+        <inertia
+            ixx="2.058-6"
+            ixy="0.0"
+            ixz="0.0"
+            iyy="2.058-6"
+            iyz="0.0"
+            izz="3.335e-6" />
+      </inertial>
+      <visual>
+        <origin
+            xyz="0 0 0"
+            rpy="0 0 0" />
+        <geometry>
+          <mesh filename="package://${MESH_FLANGE}" />
+        </geometry>
+      </visual>
+      <collision>
+        <origin
+            xyz="0 0 0"
+            rpy="0 0 0" />
+        <geometry>
+          <mesh filename="package://${MESH_FLANGE}" />
         </geometry>
       </collision>
@@ -519,8 +532,8 @@
         type="revolute">
       <origin
-          xyz="0 0 ${-70.0 * const.SCALE_MM}"
+          xyz="0 0 ${(-70.0 - 14.0) * const.SCALE_MM}"
           rpy="0 0 0" />
       <parent link="${prefix}mg400_link5" />
-      <child link="${prefix}mg400_end_effector_shaft" />
+      <child link="${prefix}mg400_end_effector_flange" />
       <axis xyz="0 0 1" />
       <limit
