Commit message: added origin

File: mg400_description/urdf/mg400.urdf.xacro (robot description, xacro)
@@ -72,4 +72,14 @@
     </collision>
   </link>
+  <joint
+      name="j0"
+      type="fixed">
+    <origin
+       xyz="-0.005 0 0.0224"
+       rpy="0 0 0" />
+    <parent link="base_link" />
+    <child link="software_origin_link" />
+  </joint>
+  <link name="software_origin_link" />
   <link name="link1">
     <inertial>

Commit message: stl -> urdf

File: mg400_description/urdf/mg400.urdf.xacro (robot description, xacro)
@@ -3,9 +3,7 @@
     xmlns:xacro="http://ros.org/wiki/xacro"
     name="mg400">
-  <!-- Import Rviz colors -->
-  <xacro:include filename="$(find mg400_description)/xacro/materials.xacro" />
   <!-- constants -->
   <xacro:include
-      filename="$(find mg400_description)/xacro/constants.xacro"
+      filename="$(find mg400_description)/urdf/common/constants.xacro"
       ns="const" />
   <!-- Base path for meshes -->
@@ -15,29 +13,35 @@
   <xacro:property
       name="MESH_BASE_LINK"
-      value="${BASE_PATH}/base_link.stl" />
+      value="${BASE_PATH}/base_link.dae" />
   <xacro:property
       name="MESH_LINK_1"
-      value="${BASE_PATH}/link1.stl" />
+      value="${BASE_PATH}/link1.dae" />
   <xacro:property
       name="MESH_LINK_2_1"
-      value="${BASE_PATH}/link2_1.stl" />
+      value="${BASE_PATH}/link2_1.dae" />
   <xacro:property
       name="MESH_LINK_2_2"
-      value="${BASE_PATH}/link2_2.stl" />
+      value="${BASE_PATH}/link2_2.dae" />
   <xacro:property
       name="MESH_LINK_3_1"
-      value="${BASE_PATH}/link3_1.stl" />
+      value="${BASE_PATH}/link3_1.dae" />
   <xacro:property
       name="MESH_LINK_3_2"
-      value="${BASE_PATH}/link3_2.stl" />
+      value="${BASE_PATH}/link3_2.dae" />
   <xacro:property
       name="MESH_LINK_4_1"
-      value="${BASE_PATH}/link4_1.stl" />
+      value="${BASE_PATH}/link4_1.dae" />
   <xacro:property
       name="MESH_LINK_4_2"
-      value="${BASE_PATH}/link4_2.stl" />
+      value="${BASE_PATH}/link4_2.dae" />
+  <xacro:property
+      name="MESH_LINK_4_3"
+      value="${BASE_PATH}/link4_3.dae" />
   <xacro:property
       name="MESH_LINK_5"
-      value="${BASE_PATH}/link5.stl" />
+      value="${BASE_PATH}/link5.dae" />
+  <xacro:property
+      name="MESH_SHAFT"
+      value="${BASE_PATH}/shaft.dae" />
   <link name="base_link">
     <inertial>
@@ -61,14 +65,5 @@
         <mesh filename="package://${MESH_BASE_LINK}" />
       </geometry>
-      <material name="white" />
-    </visual>
-    <collision>
-      <origin
-          xyz="0 0 0"
-          rpy="0 0 0" />
-      <geometry>
-        <mesh filename="package://${MESH_BASE_LINK}" />
-      </geometry>
-    </collision>
+    </visual>
   </link>
   <joint
@@ -76,6 +71,6 @@
       type="fixed">
     <origin
-       xyz="-0.005 0 0.224"
-       rpy="0 0 0" />
+        xyz="-0.005 0 0.224"
+        rpy="0 0 0" />
     <parent link="base_link" />
     <child link="software_origin_link" />
@@ -103,14 +98,5 @@
         <mesh filename="package://${MESH_LINK_1}" />
       </geometry>
-      <material name="grey" />
-    </visual>
-    <collision>
-      <origin
-          xyz="0 0 0"
-          rpy="0 0 0" />
-      <geometry>
-        <mesh filename="package://${MESH_LINK_1}" />
-      </geometry>
-    </collision>
+    </visual>
   </link>
   <joint
@@ -150,14 +136,5 @@
         <mesh filename="package://${MESH_LINK_2_1}" />
       </geometry>
-      <material name="black" />
-    </visual>
-    <collision>
-      <origin
-          xyz="0 0 0"
-          rpy="0 0 0" />
-      <geometry>
-        <mesh filename="package://${MESH_LINK_2_1}" />
-      </geometry>
-    </collision>
+    </visual>
   </link>
   <joint
@@ -197,14 +174,5 @@
         <mesh filename="package://${MESH_LINK_3_1}" />
       </geometry>
-      <material name="black" />
-    </visual>
-    <collision>
-      <origin
-          xyz="0 0 0"
-          rpy="0 0 0" />
-      <geometry>
-        <mesh filename="package://${MESH_LINK_3_1}" />
-      </geometry>
-    </collision>
+    </visual>
   </link>
   <joint
@@ -244,14 +212,5 @@
         <mesh filename="package://${MESH_LINK_4_1}" />
       </geometry>
-      <material name="white" />
-    </visual>
-    <collision>
-      <origin
-          xyz="0 0 0"
-          rpy="0 0 0" />
-      <geometry>
-        <mesh filename="package://${MESH_LINK_4_1}" />
-      </geometry>
-    </collision>
+    </visual>
   </link>
   <joint
@@ -269,4 +228,23 @@
         effort="0"
         velocity="0" />
+  </joint>
+  <link name="link4_3">
+    <visual>
+      <origin
+          xyz="0 0 0"
+          rpy="0 0 0" />
+      <geometry>
+        <mesh filename="package://${MESH_LINK_4_3}" />
+      </geometry>
+    </visual>
+  </link>
+  <joint
+      name="j4_3"
+      type="fixed">
+    <origin
+        xyz="0 0 ${2 * const.SCALE_MM}"
+        rpy="0 0 0" />
+    <parent link="link5" />
+    <child link="link4_3" />
   </joint>
   <link name="link5">
@@ -291,14 +269,5 @@
         <mesh filename="package://${MESH_LINK_5}" />
       </geometry>
-      <material name="grey" />
-    </visual>
-    <collision>
-      <origin
-          xyz="0 0 0"
-          rpy="0 0 0" />
-      <geometry>
-        <mesh filename="package://${MESH_LINK_5}" />
-      </geometry>
-    </collision>
+    </visual>
   </link>
   <joint
@@ -306,9 +275,8 @@
       type="fixed">
     <origin
-        xyz="0.0659996239003897 0.0170000000000371 0.031000800715573"
+        xyz="0.066 0.017 0.031"
         rpy="0 0 0" />
     <parent link="link4_1" />
     <child link="link5" />
-    <axis xyz="0 0 1" />
   </joint>
   <link name="end_effector_shaft">
@@ -316,11 +284,8 @@
       <origin
           xyz="0 0 0"
-          rpy="0 0 0" />
-      <geometry>
-        <cylinder
-            radius="${4.0 * const.SCALE_MM}"
-            length="${15.0 * const.SCALE_MM}" />
-      </geometry>
-      <material name="red" />
+          rpy="${180.0 * const.TO_RADIAN} 0 0" />
+      <geometry>
+        <mesh filename="package://${MESH_SHAFT}" />
+      </geometry>
     </visual>
     <collision>
@@ -371,14 +336,5 @@
         <mesh filename="package://${MESH_LINK_2_2}" />
       </geometry>
-      <material name="white" />
-    </visual>
-    <collision>
-      <origin
-          xyz="0 0 0"
-          rpy="0 0 0" />
-      <geometry>
-        <mesh filename="package://${MESH_LINK_2_2}" />
-      </geometry>
-    </collision>
+    </visual>
   </link>
   <joint
@@ -418,14 +374,5 @@
         <mesh filename="package://${MESH_LINK_3_2}" />
       </geometry>
-      <material name="black" />
-    </visual>
-    <collision>
-      <origin
-          xyz="0 0 0"
-          rpy="0 0 0" />
-      <geometry>
-        <mesh filename="package://${MESH_LINK_3_2}" />
-      </geometry>
-    </collision>
+    </visual>
   </link>
   <joint
@@ -465,14 +412,5 @@
         <mesh filename="package://${MESH_LINK_4_2}" />
       </geometry>
-      <material name="white" />
-    </visual>
-    <collision>
-      <origin
-          xyz="0 0 0"
-          rpy="0 0 0" />
-      <geometry>
-        <mesh filename="package://${MESH_LINK_4_2}" />
-      </geometry>
-    </collision>
+    </visual>
   </link>
   <joint

Commit message: fix mg400 urdf to enabale importable for other packages

File: mg400_description/urdf/mg400.urdf.xacro (robot description, xacro)
@@ -3,429 +3,13 @@
     xmlns:xacro="http://ros.org/wiki/xacro"
     name="mg400">
-  <!-- constants -->
-  <xacro:include
-      filename="$(find mg400_description)/urdf/common/constants.xacro"
-      ns="const" />
-  <!-- Base path for meshes -->
-  <xacro:property
-      name="BASE_PATH"
-      value="mg400_description/meshes" />
-  <xacro:property
-      name="MESH_BASE_LINK"
-      value="${BASE_PATH}/base_link.dae" />
-  <xacro:property
-      name="MESH_LINK_1"
-      value="${BASE_PATH}/link1.dae" />
-  <xacro:property
-      name="MESH_LINK_2_1"
-      value="${BASE_PATH}/link2_1.dae" />
-  <xacro:property
-      name="MESH_LINK_2_2"
-      value="${BASE_PATH}/link2_2.dae" />
-  <xacro:property
-      name="MESH_LINK_3_1"
-      value="${BASE_PATH}/link3_1.dae" />
-  <xacro:property
-      name="MESH_LINK_3_2"
-      value="${BASE_PATH}/link3_2.dae" />
-  <xacro:property
-      name="MESH_LINK_4_1"
-      value="${BASE_PATH}/link4_1.dae" />
-  <xacro:property
-      name="MESH_LINK_4_2"
-      value="${BASE_PATH}/link4_2.dae" />
-  <xacro:property
-      name="MESH_LINK_4_3"
-      value="${BASE_PATH}/link4_3.dae" />
-  <xacro:property
-      name="MESH_LINK_5"
-      value="${BASE_PATH}/link5.dae" />
-  <xacro:property
-      name="MESH_SHAFT"
-      value="${BASE_PATH}/shaft.dae" />
-  <link name="base_link">
-    <inertial>
-      <origin
-          xyz="0.000600637001378879 -2.53487071137343E-07 0.0560927888040551"
-          rpy="0 0 0" />
-      <mass value="3.62164811695094" />
-      <inertia
-          ixx="0.0126582175296405"
-          ixy="6.66832041405407E-08"
-          ixz="-3.52548281362717E-06"
-          iyy="0.0145891535260188"
-          iyz="5.15901657460475E-08"
-          izz="0.0195045116656827" />
-    </inertial>
-    <visual>
-      <origin
-          xyz="0 0 0"
-          rpy="0 0 0" />
-      <geometry>
-        <mesh filename="package://${MESH_BASE_LINK}" />
-      </geometry>
-    </visual>
-  </link>
-  <joint
-      name="j0"
-      type="fixed">
+  <xacro:include filename="$(find mg400_description)/urdf/mg400.xacro" />
+  <!-- links -->
+  <link name="base_link" />
+  <xacro:mg400
+      parent="base_link"
+      prefix="">
     <origin
-        xyz="-0.005 0 0.224"
+        xyz="0 0 0"
         rpy="0 0 0" />
-    <parent link="base_link" />
-    <child link="software_origin_link" />
-  </joint>
-  <link name="software_origin_link" />
-  <link name="link1">
-    <inertial>
-      <origin
-          xyz="-0.0046209286967387 -6.88107982318643E-05 0.0709919358465827"
-          rpy="0 0 0" />
-      <mass value="1.77056222753813" />
-      <inertia
-          ixx="0.00605885293080088"
-          ixy="0.000156081820035162"
-          ixz="-0.00021785654850453"
-          iyy="0.00579381982249127"
-          iyz="6.20876898015621E-05"
-          izz="0.00741058257251941" />
-    </inertial>
-    <visual>
-      <origin
-          xyz="0 0 0"
-          rpy="0 0 0" />
-      <geometry>
-        <mesh filename="package://${MESH_LINK_1}" />
-      </geometry>
-    </visual>
-  </link>
-  <joint
-      name="j1"
-      type="revolute">
-    <origin
-        xyz="${-5.0 * const.SCALE_MM} 0 ${109 * const.SCALE_MM}"
-        rpy="0 0 0" />
-    <parent link="base_link" />
-    <child link="link1" />
-    <axis xyz="0 0 1" />
-    <limit
-        lower="${-180.0 * const.TO_RADIAN}"
-        upper="${180.0 * const.TO_RADIAN}"
-        effort="0"
-        velocity="0" />
-  </joint>
-  <link name="link2_1">
-    <inertial>
-      <origin
-          xyz="-0.00321788524756698 0.0352926570826593 0.0596131328734945"
-          rpy="0 0 0" />
-      <mass value="0.0866115884541459" />
-      <inertia
-          ixx="0.000338551627157209"
-          ixy="-2.78858228577314E-09"
-          ixz="1.05212346076681E-05"
-          iyy="0.000307789653713489"
-          iyz="-1.36109590152488E-06"
-          izz="3.89949940178023E-05" />
-    </inertial>
-    <visual>
-      <origin
-          xyz="0 0 0"
-          rpy="0 0 0" />
-      <geometry>
-        <mesh filename="package://${MESH_LINK_2_1}" />
-      </geometry>
-    </visual>
-  </link>
-  <joint
-      name="j2_1"
-      type="revolute">
-    <origin
-        xyz="0.0435007595118091 -0.0357748756218899 0.118995682641123"
-        rpy="0 0 0" />
-    <parent link="link1" />
-    <child link="link2_1" />
-    <axis xyz="0 1 0" />
-    <limit
-        lower="-3.14"
-        upper="3.14"
-        effort="0"
-        velocity="0" />
-  </joint>
-  <link name="link3_1">
-    <inertial>
-      <origin
-          xyz="0.0821679417596488 0.000113044685842874 -0.00333758753063973"
-          rpy="0 0 0" />
-      <mass value="0.0375214831045061" />
-      <inertia
-          ixx="2.54761091812684E-06"
-          ixy="3.73102654491378E-07"
-          ixz="-2.02625705871199E-06"
-          iyy="0.000164234314177935"
-          iyz="-1.44731096825347E-08"
-          izz="0.000164331500854172" />
-    </inertial>
-    <visual>
-      <origin
-          xyz="0 0 0"
-          rpy="0 0 0" />
-      <geometry>
-        <mesh filename="package://${MESH_LINK_3_1}" />
-      </geometry>
-    </visual>
-  </link>
-  <joint
-      name="j3_1"
-      type="revolute">
-    <origin
-        xyz="-0.0010512570171516 0.0357748756218898 0.175001164344716"
-        rpy="0 0 0" />
-    <parent link="link2_1" />
-    <child link="link3_1" />
-    <axis xyz="0 1 0" />
-    <limit
-        lower="-3.14"
-        upper="3.14"
-        effort="0"
-        velocity="0" />
-  </joint>
-  <link name="link4_1">
-    <inertial>
-      <origin
-          xyz="0.0387878182928232 0.0170848333998282 -0.0024610990490942"
-          rpy="0 0 0" />
-      <mass value="0.0628979533925801" />
-      <inertia
-          ixx="4.78483605712844E-05"
-          ixy="1.42081909356751E-07"
-          ixz="8.32917079044309E-06"
-          iyy="5.42362047732042E-05"
-          iyz="-2.90608446019989E-08"
-          izz="3.36120409842199E-05" />
-    </inertial>
-    <visual>
-      <origin
-          xyz="0 0 0"
-          rpy="0 0 0" />
-      <geometry>
-        <mesh filename="package://${MESH_LINK_4_1}" />
-      </geometry>
-    </visual>
-  </link>
-  <joint
-      name="j4_1"
-      type="revolute">
-    <origin
-        xyz="0.174969784055705 -0.0170000000000335 0.00325187137614585"
-        rpy="0 0 0" />
-    <parent link="link3_1" />
-    <child link="link4_1" />
-    <axis xyz="0 1 0" />
-    <limit
-        lower="-3.14"
-        upper="3.14"
-        effort="0"
-        velocity="0" />
-  </joint>
-  <link name="link4_3">
-    <visual>
-      <origin
-          xyz="0 0 0"
-          rpy="0 0 0" />
-      <geometry>
-        <mesh filename="package://${MESH_LINK_4_3}" />
-      </geometry>
-    </visual>
-  </link>
-  <joint
-      name="j4_3"
-      type="fixed">
-    <origin
-        xyz="0 0 ${2 * const.SCALE_MM}"
-        rpy="0 0 0" />
-    <parent link="link5" />
-    <child link="link4_3" />
-  </joint>
-  <link name="link5">
-    <inertial>
-      <origin
-          xyz="4.24246458685662E-07 3.08507851181768E-14 -0.0349688816440933"
-          rpy="0 0 0" />
-      <mass value="0.0965276919819365" />
-      <inertia
-          ixx="4.98589992160928E-05"
-          ixy="-1.534865545378E-12"
-          ixz="3.46424449605658E-10"
-          iyy="4.98589881725446E-05"
-          iyz="-5.64890953414983E-17"
-          izz="2.130463008359E-05" />
-    </inertial>
-    <visual>
-      <origin
-          xyz="0 0 0"
-          rpy="0 0 0" />
-      <geometry>
-        <mesh filename="package://${MESH_LINK_5}" />
-      </geometry>
-    </visual>
-  </link>
-  <joint
-      name="j5_1"
-      type="fixed">
-    <origin
-        xyz="0.066 0.017 0.031"
-        rpy="0 0 0" />
-    <parent link="link4_1" />
-    <child link="link5" />
-  </joint>
-  <link name="end_effector_shaft">
-    <visual>
-      <origin
-          xyz="0 0 0"
-          rpy="${180.0 * const.TO_RADIAN} 0 0" />
-      <geometry>
-        <mesh filename="package://${MESH_SHAFT}" />
-      </geometry>
-    </visual>
-    <collision>
-      <origin
-          xyz="0 0 0"
-          rpy="0 0 0" />
-      <geometry>
-        <cylinder
-            radius="${4.0 * const.SCALE_MM}"
-            length="${15.0 * const.SCALE_MM}" />
-      </geometry>
-    </collision>
-  </link>
-  <joint
-      name="j5"
-      type="revolute">
-    <origin
-        xyz="0 0 ${-70.0 * const.SCALE_MM}"
-        rpy="0 0 0" />
-    <parent link="link5" />
-    <child link="end_effector_shaft" />
-    <axis xyz="0 0 1" />
-    <limit
-        lower="${-180.0 * const.TO_RADIAN}"
-        upper="${180.0 * const.TO_RADIAN}"
-        effort="0"
-        velocity="0" />
-  </joint>
-  <link name="link2_2">
-    <inertial>
-      <origin
-          xyz="-0.0201111131723385 0.0304999635268521 0.073632809340276"
-          rpy="0 0 0" />
-      <mass value="0.0662546292985346" />
-      <inertia
-          ixx="0.000218973873589181"
-          ixy="3.0147933007673E-10"
-          ixz="2.51402553227571E-06"
-          iyy="0.000200510070261609"
-          iyz="-1.41837669904595E-09"
-          izz="3.74316777806776E-05" />
-    </inertial>
-    <visual>
-      <origin
-          xyz="0 0 0"
-          rpy="0 0 0" />
-      <geometry>
-        <mesh filename="package://${MESH_LINK_2_2}" />
-      </geometry>
-    </visual>
-  </link>
-  <joint
-      name="j2_2"
-      type="revolute">
-    <origin
-        xyz="0.00452885682964267 -0.0305 0.141500000000001"
-        rpy="0 0 0" />
-    <parent link="link1" />
-    <child link="link2_2" />
-    <axis xyz="0 1 0" />
-    <limit
-        lower="-3.14"
-        upper="3.14"
-        effort="0"
-        velocity="0" />
-  </joint>
-  <link name="link3_2">
-    <inertial>
-      <origin
-          xyz="0.0338566736074436 0.0240208873857428 0.00452229895926692"
-          rpy="0 0 0" />
-      <mass value="0.0366692789294813" />
-      <inertia
-          ixx="7.24011830695354E-06"
-          ixy="7.93542746250724E-10"
-          ixz="-1.69163254472566E-06"
-          iyy="2.34967008246727E-05"
-          iyz="4.55507111386579E-10"
-          izz="1.66831643179488E-05" />
-    </inertial>
-    <visual>
-      <origin
-          xyz="0 0 0"
-          rpy="0 0 0" />
-      <geometry>
-        <mesh filename="package://${MESH_LINK_3_2}" />
-      </geometry>
-    </visual>
-  </link>
-  <joint
-      name="j3_2"
-      type="revolute">
-    <origin
-        xyz="-0.00105049750546494 0.00649999999999986 0.174996846985851"
-        rpy="0 0 0" />
-    <parent link="link2_2" />
-    <child link="link3_2" />
-    <axis xyz="0 1 0" />
-    <limit
-        lower="-3.14"
-        upper="3.14"
-        effort="0"
-        velocity="0" />
-  </joint>
-  <link name="link4_2">
-    <inertial>
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
Commit message: fix descirption

File: mg400_description/urdf/mg400.urdf.xacro (robot description, xacro)
@@ -4,8 +4,15 @@
     name="mg400">
   <xacro:include filename="$(find mg400_description)/urdf/mg400.xacro" />
+  <!-- arguments -->
+  <xacro:arg
+      name="prefix"
+      default="" />
+  <xacro:arg
+      name="use_arm"
+      default="True" />
   <!-- links -->
-  <link name="base_link" />
+  <link name="$(arg prefix)arm_frame_link_offset" />
   <xacro:mg400
-      parent="base_link"
+      parent="$(arg prefix)arm_frame_link_offset"
       prefix="">
     <origin

Commit message: update mesh file, launch files and urdf

File: mg400_description/urdf/mg400.urdf.xacro (robot description, xacro)
@@ -1,22 +1,26 @@
 <?xml version="1.0" encoding="utf-8"?>
 <robot
-    xmlns:xacro="http://ros.org/wiki/xacro"
-    name="mg400">
-  <xacro:include filename="$(find mg400_description)/urdf/mg400.xacro" />
-  <!-- arguments -->
-  <xacro:arg
-      name="prefix"
-      default="" />
-  <xacro:arg
-      name="use_arm"
-      default="True" />
-  <!-- links -->
-  <link name="$(arg prefix)arm_frame_link_offset" />
-  <xacro:mg400
-      parent="$(arg prefix)arm_frame_link_offset"
-      prefix="$(arg prefix)">
-    <origin
-        xyz="0 0 0"
-        rpy="0 0 0" />
-  </xacro:mg400>
+        xmlns:xacro="http://ros.org/wiki/xacro"
+        name="mg400">
+    <xacro:include filename="$(find mg400_description)/urdf/mg400.xacro" />
+    <!-- arguments -->
+    <xacro:arg
+            name="prefix"
+            default="" />
+    <xacro:arg
+            name="use_arm"
+            default="True" />
+    <xacro:arg
+            name="workspace_visible"
+            default="false" />
+    <!-- links -->
+    <link name="$(arg prefix)arm_frame_link_offset" />
+    <xacro:mg400
+            parent="$(arg prefix)arm_frame_link_offset"
+            prefix="$(arg prefix)"
+            workspace_visible="$(arg workspace_visible)">
+        <origin
+                xyz="0 0 0"
+                rpy="0 0 0" />
+    </xacro:mg400>
 </robot>

File: mg400_description/urdf/mg400.xacro (robot description, xacro)
@@ -42,7 +42,13 @@
       name="MESH_FLANGE"
       value="${BASE_PATH}/flange.dae" />
+  <xacro:property
+      name="MESH_WORKSPACE"
+      value="${BASE_PATH}/workspace.dae" />
   <xacro:macro
       name="mg400"
-      params="prefix parent *origin">
+      params="prefix parent *origin workspace_visible">
+    <material name="${prefix}mg400_workspace_material">
+      <color rgba="0.2 0.0 0.0 0.5" />
+    </material>
     <!-- links -->
     <link name="${prefix}mg400_base_link">
@@ -388,4 +394,17 @@
       </collision>
     </link>
+    <xacro:if value="${workspace_visible}">
+      <link name="${prefix}mg400_workspace">
+        <visual>
+          <origin
+              xyz="0 0 0"
+              rpy="0 0 0" />
+          <geometry>
+            <mesh filename="package://${MESH_WORKSPACE}" />
+          </geometry>
+          <material name="${prefix}mg400_workspace_material" />
+        </visual>
+      </link>
+    </xacro:if>
     <!-- joints -->
     <joint
@@ -396,4 +415,15 @@
       <xacro:insert_block name="origin" />
     </joint>
+    <xacro:if value="${workspace_visible}">
+      <joint
+          name="${prefix}workspace_joint"
+          type="fixed">
+        <origin
+            xyz="-0.005 0 0.228"
+            rpy="0 0 0" />
+        <parent link="${prefix}mg400_base_link" />
+        <child link="${prefix}mg400_workspace" />
+      </joint>
+    </xacro:if>
     <joint
         name="${prefix}mg400_j0"
