Commit message: init

File: mg400_description/urdf/mg400.urdf.xacro (robot description, xacro)
@@ -9,5 +9,5 @@
             default="" />
     <xacro:arg
-            name="use_arm"
+            name="use_single_path_arm"
             default="True" />
     <xacro:arg
@@ -15,7 +15,7 @@
             default="false" />
     <!-- links -->
-    <link name="$(arg prefix)arm_frame_link_offset" />
+    <link name="$(arg prefix)base_link" />
     <xacro:mg400
-            parent="$(arg prefix)arm_frame_link_offset"
+            parent="$(arg prefix)base_link"
             prefix="$(arg prefix)"
             workspace_visible="$(arg workspace_visible)">

File: mg400_description/urdf/mg400.xacro (robot description, xacro)
@@ -1,3 +1,8 @@
 <?xml version="1.0" encoding="UTF-8"?>
+<!--
+This file is based on MG400_ROS2's URDF file, and with some modifications related to mimic joints
+to enable MoveIt2 to handle the parallel link arm. Also, joint limits are set to avoid hitting unit
+frame.
+-->
 <robot xmlns:xacro="http://ros.org/wiki/xacro">
   <!-- constants -->
@@ -270,4 +275,5 @@
       </collision>
     </link>
+    <link name="${prefix}mg400_link4_1_virtual"></link>
     <link name="${prefix}mg400_link4_2">
       <inertial>
@@ -301,4 +307,5 @@
       </collision>
     </link>
+    <link name="${prefix}mg400_link4_2_virtual"></link>
     <link name="${prefix}mg400_link4_3">
       <inertial>
@@ -479,4 +486,7 @@
           effort="0"
           velocity="0" />
+      <mimic
+        joint="${prefix}mg400_j2_1"
+        multiplier="1.0" />
     </joint>
     <joint
@@ -509,4 +519,7 @@
           effort="0"
           velocity="0" />
+      <mimic
+        joint="${prefix}mg400_j2_1"
+        multiplier="-1.0" />
     </joint>
     <joint
@@ -517,4 +530,22 @@
           rpy="0 0 0" />
       <parent link="${prefix}mg400_link3_1" />
+      <child link="${prefix}mg400_link4_1_virtual" />
+      <axis xyz="0 1 0" />
+      <limit
+          lower="-3.14"
+          upper="3.14"
+          effort="0"
+          velocity="0" />
+      <mimic
+        joint="${prefix}mg400_j2_1"
+        multiplier="-1.0" />
+    </joint>
+    <joint
+        name="${prefix}mg400_j4_1_virtual"
+        type="revolute">
+      <origin
+          xyz="0 0 0"
+          rpy="0 0 0" />
+      <parent link="${prefix}mg400_link4_1_virtual" />
       <child link="${prefix}mg400_link4_1" />
       <axis xyz="0 1 0" />
@@ -524,4 +555,7 @@
           effort="0"
           velocity="0" />
+      <mimic
+        joint="${prefix}mg400_j3_1"
+        multiplier="-1.0" />
     </joint>
     <joint
@@ -532,4 +566,22 @@
           rpy="0 0 0" />
       <parent link="${prefix}mg400_link3_2" />
+      <child link="${prefix}mg400_link4_2_virtual" />
+      <axis xyz="0 1 0" />
+      <limit
+          lower="-3.14"
+          upper="3.14"
+          effort="0"
+          velocity="0" />
+      <mimic
+        joint="${prefix}mg400_j2_1"
+        multiplier="1.0" />
+    </joint>
+    <joint
+        name="${prefix}mg400_j4_2_virtual"
+        type="revolute">
+      <origin
+          xyz="0 0 0"
+          rpy="0 0 0" />
+      <parent link="${prefix}mg400_link4_2_virtual" />
       <child link="${prefix}mg400_link4_2" />
       <axis xyz="0 1 0" />
@@ -539,4 +591,7 @@
           effort="0"
           velocity="0" />
+      <mimic
+        joint="${prefix}mg400_j3_1"
+        multiplier="1.0" />
     </joint>
     <joint
